Commit message: convex mesh generation

File: urdf/urdf/LRMate-200iD.urdf (robot description, URDF)
Before this commit: robot LRMate-200iD, 7 links, 6 joints
Links:
- link Base: geometry collision mesh filename=package://LRMate-200iD/meshes/base.stl; visual mesh filename=package://LRMate-200iD/meshes/base.stl
- link J1: geometry collision mesh filename=package://LRMate-200iD/meshes/j1.stl; visual mesh filename=package://LRMate-200iD/meshes/j1.stl
- link J2: geometry collision mesh filename=package://LRMate-200iD/meshes/j2.stl; visual mesh filename=package://LRMate-200iD/meshes/j2.stl
- link J3: geometry collision mesh filename=package://LRMate-200iD/meshes/j3.stl; visual mesh filename=package://LRMate-200iD/meshes/j3.stl
- link J4: geometry collision mesh filename=package://LRMate-200iD/meshes/j4.stl; visual mesh filename=package://LRMate-200iD/meshes/j4.stl
- link J5: geometry collision mesh filename=package://LRMate-200iD/meshes/j5.stl; visual mesh filename=package://LRMate-200iD/meshes/j5.stl
- link J6: geometry collision mesh filename=package://LRMate-200iD/meshes/j6.stl; visual mesh filename=package://LRMate-200iD/meshes/j6.stl
